Commit message: CCoMaMergeManipulatorsUpdate

File: Examples/merge_example_manipulator.urdf (robot description, URDF)
Before this commit: robot advancedbot, 31 links, 30 joints
Links:
- link link_2_x: geometry collision sphere radius=0.05000000000000001; visual sphere radius=0.05000000000000001
- link link_2_y: geometry collision sphere radius=0.05000000000000001; visual sphere radius=0.05000000000000001
- link link_3_x: geometry collision sphere radius=0.049999999999999996; visual sphere radius=0.049999999999999996
- link link_3_y: geometry collision sphere radius=0.049999999999999996; visual sphere radius=0.049999999999999996
